File: cartridge-pmod.kicad_pcb (KiCad board)
At the start: 2 copper layers, 30.7 x 20 mm, 15 parts, among them J1 2.54-2*6P Bend insert, J2 CONFIG, U1 W25Q128JVSIM, U2 878-APS6404L-3SQR-SN, U3 878-APS6404L-3SQR-SN

Commit message: PCB layout complete: audio extension placed and routed, DRC at baseline
Board extended 30.8->56.3mm for the audio section; jack at new right edge.
PSRAM B removed (its dangling copper pruned), audio chain placed in three
rows and fully routed on F.Cu; PMOD8 reuses the original CS2 B.Cu corridor
and ducks under the +3.3V column; SCK rerouted after the PSRAM-B stub
pruning cut it (taps PMOD4 B.Cu, via, F.Cu snake past U1.5). GND pours
cover the extension on both layers with stitch vias; +3.3V zone restored
to its original comb shape with a widened top column. DRC: 0 unconnected,
errors identical to upstream qspi-pmod baseline (CONFIG jumper cut-traces
+ one pre-existing starved thermal).

Co-Authored-By: Claude Fable 5 <noreply@anthropic.com>
Claude-Session: https://claude.ai/code/session_01Xe5NzHvb72amxJFhr7WjZC
Parts:
- removed C3: 100n, Capacitor_SMD:C_0402_1005Metric
- removed C4: 1u, Capacitor_SMD:C_0402_1005Metric
- removed U3: 878-APS6404L-3SQR-SN, Package_SO:SOP-8_3.9x4.9mm_P1.27mm
- added C10: 100nF, C_0603_1608Metric, F.Cu at (179.5, 79.4)
- added C11: 47nF, C_0603_1608Metric, F.Cu at (172.4, 82.6)
- added C12: 100nF, C_0603_1608Metric, F.Cu at (175.4, 82.6)
- added C13: 47uF, C_0805_2012Metric, F.Cu at (172.8, 85.5)
- added C8: 10uF, C_0805_2012Metric, F.Cu at (176.4, 75.9)
- added C9: 100nF, C_0603_1608Metric, F.Cu at (179.6, 75.9)
- added J3: PJ-320B, BOOMELE_PJ-320B, F.Cu at (187.7, 84.7)
- added L1: MLF2012-3R3K, L_0805_2012Metric, F.Cu at (172.6, 75.9)
- added R4: 120R, R_0603_1608Metric, F.Cu at (176.2, 79.4)
- added R5: 33R, R_0603_1608Metric, F.Cu at (178.4, 82.6)
- added R6: 470R, R_0603_1608Metric, F.Cu at (176.4, 85.5)
- added RV1: 3362P-1-201LF, TRIM_3362P-1-102, F.Cu at (175.0, 90.7)
- added U4: 74LVCE1G126SE-7, SOT-353_SC-70-5, F.Cu at (172.8, 79.4)
Routing:
- net AUDIO_OUT: track 0.00 -> 23.9 mm
- net AUDIO_N2: track 0.00 -> 19.1 mm
- net AUDIO_N1: track 0.00 -> 15.7 mm
- net AUDIO_VCCA: track 0.00 -> 12.9 mm
- net PMOD6: track 69.1 -> 58.7 mm
- net PMOD8: track 18.9 -> 27.7 mm, vias 1 -> 3
- net PMOD5: track 36.6 -> 30.6 mm, vias 3 -> 2
- net PMOD3: track 39.5 -> 35.3 mm
- net PMOD4: track 37.1 -> 34.1 mm, vias 1 -> 2
- net AUDIO_BUF: track 0.00 -> 2.41 mm
- net +3.3V: track 12.5 -> 14.8 mm
- net PMOD2: track 43.6 -> 42.2 mm, vias 3 -> 2
- net GND: track 13.5 -> 14.7 mm, vias 7 -> 15
- added copper zone on F.Cu, net GND
Other:
- board size 30.7 x 20 mm -> 56 x 20 mm
