File: cartridge-pmod.kicad_pcb (KiCad board)
At the start: 2 copper layers, 56 x 20 mm, 25 parts, among them J1 2.54-2*6P Bend insert, J2 CONFIG, J3 PJ-320B, U1 W25Q128JVSIM, U2 878-APS6404L-3SQR-SN, U4 74LVCE1G126SE-7

Commit message: Pearto mascot on back silkscreen; fix stale PSRAM B CS jumper label
Logo traced from pearto.jpeg (white background flood-removed, pear/hood
outlines Moore-traced + RDP-simplified, eyes/mouth as parametric circles),
8.6mm tall on B.Silkscreen above the jack anchors, X-mirrored for correct
back-side viewing. Jumper legend for uio7 now reads AUDIO. DRC unchanged.

Co-Authored-By: Claude Fable 5 <noreply@anthropic.com>
Claude-Session: https://claude.ai/code/session_01Xe5NzHvb72amxJFhr7WjZC
Other:
- board text added: "AUDIO"
- board text removed: "PSRAM B CS"
Changed lines of the file:
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@@
 		(layer "F.SilkS")
+	)
+	(gr_poly
+		(pts
+			(xy 188.840201 75.604187) (xy 188.768174 75.618592) (xy 188.667336 75.748241) (xy 188.508877 76.137185)
+			(xy 188.364824 76.698994) (xy 188.422445 76.771021) (xy 188.566499 76.670184) (xy 188.739363 76.108375)
+			(xy 188.969849 75.863484) (xy 188.941038 75.661809)
+		)
+		(stroke
+			(width 0.16)
+			(type default)
+		)
+		(fill no)
+		(layer "B.SilkS")
+	)
+	(gr_poly
+		(pts
+			(xy 188.465661 78.643718) (xy 188.206365 78.715745) (xy 188.062311 78.830988) (xy 187.975879 78.787772)
+			(xy 187.947068 78.888609) (xy 187.81742 78.960636) (xy 187.759798 79.090284) (xy 187.687772 79.047068)
+			(xy 187.327638 79.407202) (xy 187.197989 79.392797) (xy 187.125963 79.53685) (xy 187.111557 79.493634)
+			(xy 186.909882 79.666499) (xy 186.852261 80.113065) (xy 186.938693 81.107035) (xy 186.996314 81.222278)
+			(xy 187.125963 81.251088) (xy 187.169179 81.510385) (xy 187.370854 81.740871) (xy 187.342043 81.755276)
+			(xy 187.60134 81.942546) (xy 187.572529 82.014572) (xy 187.486097 82.043383) (xy 187.730988 82.317085)
+			(xy 188.566499 82.345896) (xy 188.667336 82.230653) (xy 188.796984 82.216247) (xy 188.998659 81.971356)
+			(xy 189.157118 81.884924) (xy 189.286767 81.683249) (xy 189.474036 81.596817) (xy 189.646901 81.395142)
+			(xy 189.704522 81.193467) (xy 189.819765 81.063819) (xy 189.906197 80.833333) (xy 190.035845 80.31474)
+			(xy 190.064656 80.141876) (xy 189.992629 79.882579) (xy 189.906197 79.652093) (xy 189.762144 79.493634)
+			(xy 189.603685 79.450418) (xy 189.358793 79.277554) (xy 189.315577 79.306365) (xy 189.21474 79.162311)
+			(xy 189.113902 79.119095) (xy 189.085092 79.032663) (xy 188.984254 79.003852) (xy 188.782579 78.787772)
+			(xy 188.62412 78.672529)
+		)
+		(stroke
+			(width 0.16)
+			(type default)
+		)
+		(fill no)
+		(layer "B.SilkS")
+	)
+	(gr_poly
+		(pts
+			(xy 188.897822 75.50335) (xy 188.739363 75.517755) (xy 188.62412 75.661809) (xy 188.393634 76.194807)
+			(xy 188.321608 76.583752) (xy 188.263986 76.670184) (xy 188.191959 76.727805) (xy 187.990284 76.742211)
+			(xy 187.644556 76.857453) (xy 187.399664 77.087939) (xy 187.212395 77.404857) (xy 187.111557 77.822613)
+			(xy 186.996314 78.038693) (xy 186.895477 78.643718) (xy 186.809045 78.715745) (xy 186.708207 78.989447)
+			(xy 186.578559 79.162311) (xy 186.290452 79.997822) (xy 186.189614 80.170686) (xy 186.175209 80.948576)
+			(xy 186.362479 81.812897) (xy 186.333668 81.956951) (xy 185.901507 82.014572) (xy 185.901507 83.498324)
+			(xy 186.103182 83.541541) (xy 186.146398 83.498324) (xy 186.189614 83.599162) (xy 186.463316 83.642378)
+			(xy 187.255611 83.613567) (xy 187.875041 83.527135) (xy 188.696147 83.311055) (xy 188.912227 83.210217)
+			(xy 189.243551 82.950921) (xy 189.344388 82.720435) (xy 189.690117 82.475544) (xy 190.323953 81.582412)
+			(xy 190.468006 81.179061) (xy 190.468006 80.415577) (xy 190.338358 79.551256) (xy 190.251926 79.378391)
+			(xy 190.02144 79.191122) (xy 189.790954 78.903015) (xy 189.574874 78.542881) (xy 189.445226 77.851423)
+			(xy 189.329983 77.678559) (xy 189.142713 77.102345) (xy 188.681742 76.7134) (xy 188.782579 76.252428)
+			(xy 189.056281 75.849078) (xy 189.02747 75.632998)
+		)
+		(stroke
+			(width 0.16)
+			(type default)
+		)
+		(fill no)
+		(layer "B.SilkS")
+	)
+	(gr_circle
+		(center 187.397335 80.255942)
+		(end 187.131774 80.255942)
+		(stroke
+			(width 0.16)
+			(type default)
+		)
+		(fill no)
+		(layer "B.SilkS")
+	)
+	(gr_circle
+		(center 187.397335 80.255942)
+		(end 187.557335 80.255942)
+		(stroke
+			(width 0.16)
+			(type default)
+		)
+		(fill yes)
+		(layer "B.SilkS")
+	)
+	(gr_circle
+		(center 188.380918 81.769785)
+		(end 188.164904 81.769785)
+		(stroke
+			(width 0.16)
+			(type default)
+		)
+		(fill yes)
+		(layer "B.SilkS")
+	)
+	(gr_circle
+		(center 189.227891 80.315532)
+		(end 188.96233 80.315532)
+		(stroke
+			(width 0.16)
+			(type default)
+		)
+		(fill no)
+		(layer "B.SilkS")
+	)
+	(gr_circle
+		(center 189.227891 80.315532)
+		(end 189.387891 80.315532)
+		(stroke
+			(width 0.16)
+			(type default)
+		)
+		(fill yes)
+		(layer "B.SilkS")
 	)
 	(gr_line
@@
 		)
 	)
-	(gr_text "PSRAM B CS"
+	(gr_text "AUDIO"
 		(at 165.5 89.2 0)
 		(layer "B.SilkS")

Commit message: Pearto v2: round belly, smile, caption; add FABRICATION.md guide
Pear/hood bottoms replaced with smooth half-ellipse belly, mouth is now a
smile arc, caption Cartridge Pmod by JA on back silk. Step-by-step JLCPCB
export+ordering guide in FABRICATION.md (Fabrication Toolkit or kicad-cli).

Co-Authored-By: Claude Fable 5 <noreply@anthropic.com>
Claude-Session: https://claude.ai/code/session_01Xe5NzHvb72amxJFhr7WjZC
Other:
- board text added: "Cartridge Pmod by JA"
Changed lines of the file:
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@@
 			(xy 187.327638 79.407202) (xy 187.197989 79.392797) (xy 187.125963 79.53685) (xy 187.111557 79.493634)
 			(xy 186.909882 79.666499) (xy 186.852261 80.113065) (xy 186.938693 81.107035) (xy 186.996314 81.222278)
-			(xy 187.125963 81.251088) (xy 187.169179 81.510385) (xy 187.370854 81.740871) (xy 187.342043 81.755276)
-			(xy 187.60134 81.942546) (xy 187.572529 82.014572) (xy 187.486097 82.043383) (xy 187.730988 82.317085)
-			(xy 188.566499 82.345896) (xy 188.667336 82.230653) (xy 188.796984 82.216247) (xy 188.998659 81.971356)
-			(xy 189.157118 81.884924) (xy 189.286767 81.683249) (xy 189.474036 81.596817) (xy 189.646901 81.395142)
+			(xy 187.125963 81.251088) (xy 187.137487 81.461407) (xy 187.169179 81.609782) (xy 187.223919 81.753835)
+			(xy 187.298827 81.889246) (xy 187.392462 82.016013) (xy 187.503383 82.129815) (xy 187.63015 82.229212)
+			(xy 187.771323 82.314204) (xy 187.921139 82.381909) (xy 188.081038 82.429447) (xy 188.2467 82.459698)
+			(xy 188.415242 82.469782) (xy 188.583785 82.459698) (xy 188.749447 82.429447) (xy 188.909346 82.381909)
+			(xy 189.059162 82.314204) (xy 189.200335 82.229212) (xy 189.327102 82.129815) (xy 189.438023 82.016013)
+			(xy 189.531658 81.889246) (xy 189.606566 81.753835) (xy 189.661306 81.609782) (xy 189.692998 81.461407)
 			(xy 189.704522 81.193467) (xy 189.819765 81.063819) (xy 189.906197 80.833333) (xy 190.035845 80.31474)
 			(xy 190.064656 80.141876) (xy 189.992629 79.882579) (xy 189.906197 79.652093) (xy 189.762144 79.493634)
@@
 			(xy 186.996314 78.038693) (xy 186.895477 78.643718) (xy 186.809045 78.715745) (xy 186.708207 78.989447)
 			(xy 186.578559 79.162311) (xy 186.290452 79.997822) (xy 186.189614 80.170686) (xy 186.175209 80.948576)
-			(xy 186.362479 81.812897) (xy 186.333668 81.956951) (xy 185.901507 82.014572) (xy 185.901507 83.498324)
-			(xy 186.103182 83.541541) (xy 186.146398 83.498324) (xy 186.189614 83.599162) (xy 186.463316 83.642378)
-			(xy 187.255611 83.613567) (xy 187.875041 83.527135) (xy 188.696147 83.311055) (xy 188.912227 83.210217)
-			(xy 189.243551 82.950921) (xy 189.344388 82.720435) (xy 189.690117 82.475544) (xy 190.323953 81.582412)
-			(xy 190.468006 81.179061) (xy 190.468006 80.415577) (xy 190.338358 79.551256) (xy 190.251926 79.378391)
-			(xy 190.02144 79.191122) (xy 189.790954 78.903015) (xy 189.574874 78.542881) (xy 189.445226 77.851423)
-			(xy 189.329983 77.678559) (xy 189.142713 77.102345) (xy 188.681742 76.7134) (xy 188.782579 76.252428)
-			(xy 189.056281 75.849078) (xy 189.02747 75.632998)
-		)
-		(stroke
-			(width 0.16)
-			(type default)
-		)
-		(fill no)
-		(layer "B.SilkS")
-	)
-	(gr_circle
-		(center 187.397335 80.255942)
-		(end 187.131774 80.255942)
+			(xy 186.193936 81.615544) (xy 186.248676 81.863316) (xy 186.337989 82.102445) (xy 186.463316 82.33005)
+			(xy 186.618894 82.538927) (xy 186.803283 82.729078) (xy 187.015041 82.89618) (xy 187.248408 83.035912)
+			(xy 187.500502 83.148274) (xy 187.765561 83.228944) (xy 188.042144 83.279363) (xy 188.321608 83.295209)
+			(xy 188.601072 83.279363) (xy 188.877654 83.228944) (xy 189.142713 83.148274) (xy 189.394807 83.035912)
+			(xy 189.628174 82.89618) (xy 189.839932 82.729078) (xy 190.024321 82.538927) (xy 190.179899 82.33005)
+			(xy 190.305226 82.102445) (xy 190.394539 81.863316) (xy 190.449279 81.615544) (xy 190.468006 81.179061)
+			(xy 190.468006 80.415577) (xy 190.338358 79.551256) (xy 190.251926 79.378391) (xy 190.02144 79.191122)
+			(xy 189.790954 78.903015) (xy 189.574874 78.542881) (xy 189.445226 77.851423) (xy 189.329983 77.678559)
+			(xy 189.142713 77.102345) (xy 188.681742 76.7134) (xy 188.782579 76.252428) (xy 189.056281 75.849078)
+			(xy 189.02747 75.632998)
+		)
 		(stroke
 			(width 0.16)
@@
 	)
 	(gr_circle
-		(center 188.380918 81.769785)
-		(end 188.164904 81.769785)
-		(stroke
-			(width 0.16)
-			(type default)
-		)
-		(fill yes)
-		(layer "B.SilkS")
-	)
-	(gr_circle
-		(center 189.227891 80.315532)
-		(end 188.96233 80.315532)
-		(stroke
-			(width 0.16)
-			(type default)
-		)
-		(fill no)
+		(center 187.397335 80.255942)
+		(end 187.662896 80.255942)
+		(stroke
+			(width 0.16)
+			(type default)
+		)
+		(fill no)
+		(layer "B.SilkS")
+	)
+	(gr_arc
+		(start 188.841889 81.699198)
+		(mid 188.380918 81.97146)
+		(end 187.919946 81.699198)
+		(stroke
+			(width 0.2)
+			(type default)
+		)
 		(layer "B.SilkS")
 	)
@@
 		)
 		(fill yes)
+		(layer "B.SilkS")
+	)
+	(gr_circle
+		(center 189.227891 80.315532)
+		(end 189.493452 80.315532)
+		(stroke
+			(width 0.16)
+			(type default)
+		)
+		(fill no)
 		(layer "B.SilkS")
 	)
@@
 		)
 	)
+	(gr_text "Cartridge Pmod by JA"
+		(at 189 88.8 0)
+		(layer "B.SilkS")
+		(effects
+			(font
+				(size 0.8 0.8)
+				(thickness 0.13)
+			)
+			(justify mirror)
+		)
+	)
